File: core/BMP388_I2C.sch (KiCad schematic (older format))
At the start: 6 parts

Commit message: added connector to core and determined pinout
Parts:
- U: renamed from U?; footprint calstar:BMP388 -> star-common-lib:BMP388; symbol calstar:BMP388 -> star-common-lib:BMP388
Changed lines of the file:
@@
 EESchema Schematic File Version 4
-LIBS:core-cache
-EELAYER 26 0
+EELAYER 30 0
 EELAYER END
 $Descr A4 11693 8268
@@
 BMP388 Hierarchical Block (I2C)
 $Comp
-L calstar:BMP388 U?
+L star-common-lib:BMP388 U?
 U 1 1 5E6D1ACA
 P 5850 4050
-F 0 "U?" H 5850 4525 50  0000 C CNN
+AR Path="/5E6D1ACA" Ref="U?"  Part="1"
+AR Path="/5E6CF5BB/5E6D1ACA" Ref="U"  Part="1"
+F 0 "U" H 5850 4525 50  0000 C CNN
 F 1 "BMP388" H 5850 4434 50  0000 C CNN
-F 2 "calstar:BMP388" H 5850 4600 50  0001 C CNN
+F 2 "star-common-lib:BMP388" H 5850 4600 50  0001 C CNN
 F 3 "" H 5850 4450 50  0001 C CNN
 	1    5850 4050
