File: core/BNO055.sch (KiCad schematic (older format))
At the start: 9 parts, among them U4 BNO055

Commit message: bump hardware-sch-blocks pre-PR
Parts:
- removed C17: 6.8nF, Capacitor_SMD:C_0603_1608Metric, symbol Device:C
- removed C18: 120nF, Capacitor_SMD:C_0603_1608Metric, symbol Device:C
- removed C19, C20: 100nF, Capacitor_SMD:C_0603_1608Metric, symbol Device:C
- removed R10, R11, R8, R9: 10k, Resistor_SMD:R_0603_1608Metric, symbol Device:R
- removed U4: BNO055, Package_LGA:LGA-28_5.2x3.8mm_P0.5mm, symbol Sensor_Motion:BNO055
Connections:
- net labels removed: +3.3V, GND, INT, SCL, SDA, nRESET
- wire segments 60 -> 0
- no-connect marks 3 -> 0
Other:
- note removed: "BNO055 Hierarchical Block (I2C)"
