File: core/core.sch (KiCad schematic (older format))
At the start: 22 parts, among them J1 Micro_SD_Card, J2 UART_DEBUG, J3 Conn_ARM_JTAG_SWD_10, J4 Conn_01x02, SW1 SW_Push, U1 AP1509-33, U2 AP1509-33

Commit message: Fixed SD card reader connection
Connections:
- net labels added: SCI3_SCK, SCI3_nSS, SPI3_MISO, SPI3_MOSI
- net labels removed: CS2, MISO2, MOSI2, SCK2, VDD
- wire segments 164 -> 172
- no-connect marks 27 -> 21
Other:
- moved on the sheet: C3, C4, C5, C6, D1, D2, F1, J2, J3, J4, JP1, L1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

Commit message: Done schematic
Parts:
- added J? (x2): CAS_stacking, symbol star-common-lib:CAS_stacking
Connections:
- net +3V3: now also J?.A35 (3.3VA), J?.A36 (3.3VB)
- net +5V: now also J?.A5 (5VA), J?.A6 (5VB)
- net +BATT: now also J?.A39 (VDD_BATTA), J?.A40 (VDD_BATTB)
- net GND: now also J?.A15 (GND5), J?.A16 (GND6), J?.A26 (GND7), J?.A3 (GND1), J?.A30 (GND8), J?.A34 (GND9), J?.A37 (GND10), J?.A38 (GND11), J?.A4 (GND2), J?.A7 (GND3), J?.A8 (GND4), J?.B1 (GND12), J?.B10 (GND18), J?.B11 (GND19), J?.B12 (GND20), J?.B3 (GND13), J?.B4 (GND14), J?.B6 (GND15), J?.B7 (GND16), J?.B8 (GND17)
- net GPIO1: now also J?.A1 (INT1)
- net GPIO2: now also J?.A2 (INT2)
- net GPIO3: now also J?.A9 (INT3)
- net GPIO4: now also J?.A10 (INT4)
- net GPIO5: now also J?.A11 (INT5)
- net GPIO6: now also J?.A12 (INT6)
- net GPIO7: now also J?.A19 (INT7)
- net GPIO8: now also J?.A20 (INT8)
- net I2C1_SCL: now also J?.A13 (I2C0_SCL)
- net I2C1_SDA: now also J?.A14 (I2C0_SDA)
- net I2C3_SCL: now also J?.A17 (I2C1_SCL)
- net I2C3_SDA: now also J?.A18 (I2C1_SDA)
- net SPI1_MISO: now also J?.B5 (SPIHS_MISO)
- net SPI1_MOSI: now also J?.B9 (SPIHS_MOSI)
- net SPI1_SCK: now also J?.B2 (SPIHS_SCK)
- net SPI1_nSS: now also J?.B13 (SPIHS_nSS1), J?.B14 (SPIHS_nSS2)
- net SPI2_MISO: now also J?.A24 (SPI0_MISO)
- net SPI2_MOSI: now also J?.A28 (SPI0_MOSI)
- net SPI2_SCK: now also J?.A32 (SPI0_SCK)
- net SPI2_nSS: now also J?.A21 (SPI0_nSS1), J?.A22 (SPI0_nSS2), J?.A23 (SPI0_nSS3), J?.A25 (SPI0_nSS4), J?.A27 (SPI0_nSS5), J?.A29 (SPI0_nSS6), J?.A31 (SPI0_nSS7), J?.A33 (SPI0_nSS8)
- no-connect marks 21 -> 47
Other:
- moved on the sheet: F1, J2, J3, J4, JP1, R1, R2, R3, SW1
