File: core/core.sch (KiCad schematic (older format))
At the start: 60 parts, among them J1 Micro_SD_Card, J2 UART_DEBUG, J3 Conn_ARM_JTAG_SWD_10, J4 Conn_01x02, J5 USB_OTG, SW1 SW_Push, SW2 SW_Push, U1 SC18IS600, U2 AP1509-33, U3 AP1509-33

Commit message: Prepare PR
Parts:
- U1: symbol SC18IS602BIPW:SC18IS600 -> core-rescue:SC18IS600-SC18IS602BIPW
Changed lines of the file:
@@
 SPI3_MISO
 $Comp
-L SC18IS602BIPW:SC18IS600 U1
+L core-rescue:SC18IS600-SC18IS602BIPW U1
 U 1 1 5F37FC88
 P 1750 5700

Commit message: Sync changes
Parts:
- added R? (x3): 1k, symbol Device:R
Connections:
- net GND: now also J5.6 (Shield), R?.2, R?.2, R?.2; no longer D1.1 (K), D2.1 (K), D5.1 (K)
- net TDI: now reaches J3.8 (NC/TDI)
- new net: D1.1 (K), R?.1
- new net: D2.1 (K), R?.1
- new net: D5.1 (K), R?.1
- no-connect marks 16 -> 12
Other:
- note added: "Note: SPIHS-nSS1 missing"
- note added: "USB"
- note added: "What to keep?"
- note removed: "Note: SPIHS-nSS2 missing"
- note removed: "PB3 is used by SWO and cannot\nbe used as SPI3_NSS2\n"
- note removed: "What am I suppose to put\nhere when I have a fuel gauge?"
- note removed: "What's JDTI?\n"
- note removed: "What's shield?\n"
- moved on the sheet: D1, D2, D5, J4, J5, JP1, R5, SW1, SW2
