File: blackpowder-ignition/blackpowder-ignition.kicad_pcb (KiCad board)
At the start: 2 copper layers, 63.5 x 63.5 mm, 43 parts, among them J1 CAS_stacking, J2 Conn_01x02, J3 Conn_01x02, J4 Conn_01x02, J5 Conn_01x02, J6 Conn_01x02, J7 Conn_01x02, J8 Conn_01x02, Q1 FDS6898A, Q2 FDS6898A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

Commit message: nicer models, finished routing
Connections:
- net A0 renamed /A0
- net A1 renamed /A1
- net A2 renamed /A2
- net igniteA renamed /igniteA
- net igniteB renamed /igniteB
- net igniteC renamed /igniteC
- net igniteD renamed /igniteD
- net igniteE renamed /igniteE
- net igniteF renamed /igniteF
- net ~contA~ renamed /~contA~
- net ~contB~ renamed /~contB~
- net ~contC~ renamed /~contC~
- net ~contD~ renamed /~contD~
- net ~contE~ renamed /~contE~
- net ~contF~ renamed /~igniteF~
